File: X17-Power-Slab-master/X17-Power-Slab-Master/powerflags.kicad_sch (KiCad schematic)
At the start: 0 parts

Commit message: Alumni Design Review Pre-Changes
No 48V to 5V Schematic, unfinished STM32 connections, DRC issues, flags not neat.
Other:
- note added: "Brick Labels"
- note added: "STM32 Labels"
