File: X17-Power-Slab-master/X17-Power-Slab-Master/_autosave-X17-Power-Slab-Master.kicad_sch (KiCad schematic)
At the start: 17 parts, among them J1 Conn_01x05, J2 ET60S-D04-3-08-D04-X-R1-S, Q1 NMOS, U1 AZ1117IH-3.3TRG1, U4 STM32F091CCTx, Y1 Crystal

Commit message: for daniel
Parts:
- removed J1: Conn_01x05, symbol Connector_Generic:Conn_01x05
- removed U4: STM32F091CCTx, Package_QFP:LQFP-48_7x7mm_P0.5mm, symbol MCU_ST_STM32F0:STM32F091CCTx
Other:
- added sheet STM32 (stm32sheet.kicad_sch)
- note added: "change schematic bc input/output diffs"
- note added: "to 12V gnd"
- note added: "to 5V gnd for digital logic"
