File: X17-Power-Slab-master/X17-Power-Slab-Master/24V_output_powerslab.kicad_sch (KiCad schematic)
At the start: 16 parts, among them Q2 PMOS

Commit message: Schematic Updates
#SlayedTheDayAway
Parts:
- renumbered 1 to 11, Iout to Iout1
Changed lines of the file:
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@@
 		(dnp no)
 		(fields_autoplaced yes)
-		(property "Reference" "Iout"
+		(property "Reference" "Iout1"
 			(at 274.32 115.5699 0)
 			(effects
@@
 			(project ""
 				(path "/57e59c68-7be1-495e-b535-e78e0f561e15/a173c630-d818-4bdf-96f3-617172bdeb8e"
-					(reference "Iout")
+					(reference "Iout1")
 					(unit 1)
 				)
@@
 		(dnp no)
 		(fields_autoplaced yes)
-		(property "Reference" "1"
+		(property "Reference" "11"
 			(at 132.08 60.96 0)
 			(effects
@@
 			(project ""
 				(path "/57e59c68-7be1-495e-b535-e78e0f561e15/a173c630-d818-4bdf-96f3-617172bdeb8e"
-					(reference "1")
+					(reference "11")
 					(unit 1)
 				)

Commit message: Schematic Full Update
Probs can start pacing after this.
Diode on RVP changed,
Button changed
Reverse voltage updated
Symbols updated to remove DRCs
GNDs changed
Connector updated
Parts:
- 11: footprint MUY08A -> (none)
- R13, R14, R15, R16, R17: footprint (none) -> Resistor_SMD:R_0603_1608Metric_Pad0.98x0.95mm_HandSolder
Changed lines of the file:
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@@
 			)
 		)
-		(property "Footprint" ""
+		(property "Footprint" "Resistor_SMD:R_0603_1608Metric_Pad0.98x0.95mm_HandSolder"
 			(at 252.476 100.584 90)
 			(effects
@@
 			)
 		)
-		(property "Footprint" ""
+		(property "Footprint" "Resistor_SMD:R_0603_1608Metric_Pad0.98x0.95mm_HandSolder"
 			(at 252.476 118.364 90)
 			(effects
@@
 			)
 		)
-		(property "Footprint" ""
+		(property "Footprint" "Resistor_SMD:R_0603_1608Metric_Pad0.98x0.95mm_HandSolder"
 			(at 196.596 74.676 90)
 			(effects
@@
 			)
 		)
-		(property "Footprint" ""
+		(property "Footprint" "Resistor_SMD:R_0603_1608Metric_Pad0.98x0.95mm_HandSolder"
 			(at 89.916 70.104 90)
 			(effects
@@
 			)
 		)
-		(property "Footprint" "MUY08A"
+		(property "Footprint" ""
 			(at 101.6 71.12 0)
 			(effects
@@
 			)
 		)
-		(property "Footprint" ""
+		(property "Footprint" "Resistor_SMD:R_0603_1608Metric_Pad0.98x0.95mm_HandSolder"
 			(at 96.266 54.356 90)
 			(effects
