File: X17-Power-Slab-master/X17-Power-Slab-Master/X17-Power-Slab-Master.kicad_pcb (KiCad board)
At the start: 2 copper layers, 302.3 x 119 mm, 62 parts, among them J2 ET60T-D04-3-08-D04-X-R1-S, J3 796636-6, J4 Conn_01x05, Q2 TSM340N06CP ROG, SW2 1825910-6, U1 AZ1117IH-3.3TRG1, U4 STM32F091CCTx, U6 MAX485E, U7 ABLS-8.000MHZ-B2-T

Commit message: Connectors and Testpoints for all components
Errors with thermal relief in my capacitors
Parts:
- moved U6 250.7 mm to (115.0, -14.9), turned to 0 degrees
- moved TP3 165.5 mm to (149.5, 130.5)
- moved TP4 151.3 mm to (116.0, 119.0)
- moved R18 148.6 mm to (75.0, 109.0), turned to 180 degrees
- moved R27 146.3 mm to (74.9, 107.0), turned to 180 degrees
- moved TP15 146.2 mm to (85.0, 120.0)
- moved TP14 143.0 mm to (85.0, 110.5)
- moved TP2 127.1 mm to (102.5, 92.0)
- moved TP5 118.7 mm to (78.0, 56.5)
- moved TP6 99.5 mm to (112.0, 61.5)
- moved TP1 86.6 mm to (145.0, 51.5)
- moved D1 4.57 mm to (131.5, 57.0), turned to -90 degrees
- moved R10 3.91 mm to (125.0, 122.5)
Connections:
- R18 pad 1: 5V_GND -> 12V_5V_GND
- TP15 pad 1: 5V_GND -> 12V_5V_GND
- U5 pad 5: 5V_GND -> 12V_5V_GND
Routing:
- net Net-(U5-Trim): track 0.00 -> 85.9 mm
- net 5V: track 0.00 -> 71.0 mm, vias 0 -> 1
- net 12V_5V_GND: track 0.00 -> 62.5 mm, vias 0 -> 1
- net 48V: track 3.17 -> 65.5 mm, vias 1 -> 5
- net Net-(U8-SA0/SA1): track 0.00 -> 20.2 mm
- net 48V_GND: track 21.9 -> 35.9 mm, vias 1 -> 0
- net RAW_48V_GND: track 18.1 -> 30.1 mm
- net Net-(D1-K): track 8.23 -> 11.3 mm

Commit message: Final Power Board
There is an error of a missing connection for two of the test points 12_5V_GND for the 5V brick and the 12V brick and I cant resolve the DRC error.
Parts:
- removed C1, C3: 10uF, Capacitor_SMD:C_0603_1608Metric_Pad1.08x0.95mm_HandSolder
- removed C10, C11, C12, C13, C18: 0.1uF, Capacitor_SMD:C_0603_1608Metric_Pad1.08x0.95mm_HandSolder
- removed C14, C15: 4.7uF, Capacitor_SMD:C_0603_1608Metric_Pad1.08x0.95mm_HandSolder
- removed C16, C17: 18pF, Capacitor_SMD:C_0603_1608Metric_Pad1.08x0.95mm_HandSolder
- removed C2: .1uF, Capacitor_SMD:C_0603_1608Metric_Pad1.08x0.95mm_HandSolder
- removed C4: 22uF, Capacitor_SMD:C_0603_1608Metric_Pad1.08x0.95mm_HandSolder
- removed D3: LED, LED_SMD:LED_0805_2012Metric_Pad1.15x1.40mm_HandSolder
- removed J4: Conn_01x05, Connector_PinHeader_2.54mm:PinHeader_1x05_P2.54mm_Vertical
- removed R2, R3, R4, R5: 10000, Resistor_SMD:R_0603_1608Metric_Pad0.98x0.95mm_HandSolder
- removed R20: 470, Resistor_SMD:R_0603_1608Metric_Pad0.98x0.95mm_HandSolder
- removed R21, R22: 4.7k, Resistor_SMD:R_0603_1608Metric_Pad0.98x0.95mm_HandSolder
- removed R26: 10k, Resistor_SMD:R_0603_1608Metric_Pad0.98x0.95mm_HandSolder
- removed R6, R7: 20000, Resistor_SMD:R_0603_1608Metric_Pad0.98x0.95mm_HandSolder
- removed R8: 120, Resistor_SMD:R_0603_1608Metric_Pad0.98x0.95mm_HandSolder
- removed SW2: 1825910-6, STM switch:SW4_1825910-B_TEC
- removed TP13, TP16: TestPoint, TestPoint:TestPoint_Pad_D4.0mm
- removed U1: AZ1117IH-3.3TRG1, AZ1117_4pin:SOT230P700X185-4N
- removed U4: STM32F091CCTx, Package_QFP:LQFP-48_7x7mm_P0.5mm
- removed U6: MAX485E, Package_SO:SOIC-8_3.9x4.9mm_P1.27mm
- removed U7: ABLS-8.000MHZ-B2-T, footprints:ABLS-8.000MHZ-B2-T_ABR
- moved TP1 5.50 mm to (150.5, 51.5)
Routing:
- net 48V_GND: track 35.9 -> 46.1 mm

Commit message: Final Board 2
See prior description
Parts:
- moved TP15 5.00 mm to (85.0, 125.0)
Routing:
- net 12V_5V_GND: track 62.5 -> 69.4 mm
Changed lines of the file:
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@@
 	(footprint "TestPoint:TestPoint_Pad_D4.0mm"
 		(layer "F.Cu")
-		(at 85 120)
+		(at 85 125)
 		(descr "SMD pad as test Point, diameter 4.0mm")
 		(tags "test point SMD pad")
@@
 	)
 	(segment
-		(start 88 120)
-		(end 92 116)
+		(start 92 113.5)
+		(end 89 116.5)
+		(width 1.27)
+		(layer "F.Cu")
+		(net 26)
+	)
+	(segment
+		(start 92 132.89)
+		(end 92 128.5)
+		(width 1.27)
+		(layer "F.Cu")
+		(net 26)
+	)
+	(segment
+		(start 92.03 132.92)
+		(end 92 132.89)
 		(width 1.27)
 		(layer "F.Cu")
@@
 	)
 	(segment
-		(start 92 123)
-		(end 90 125)
+		(start 92 106)
+		(end 92 113.5)
 		(width 1.27)
 		(layer "F.Cu")
@@
 	(segment
 		(start 92 128.5)
-		(end 92 132.89)
+		(end 90 126.5)
 		(width 1.27)
 		(layer "F.Cu")
@@
 	)
 	(segment
-		(start 92 106)
-		(end 92 116)
+		(start 87 116.5)
+		(end 85 118.5)
 		(width 1.27)
 		(layer "F.Cu")
@@
 	)
 	(segment
-		(start 90 125)
-		(end 90 126.5)
-		(width 1.27)
+		(start 82.5 102.5)
+		(end 76 109)
+		(width 0.762)
 		(layer "F.Cu")
 		(net 26)
 	)
 	(segment
-		(start 85 120)
-		(end 88 120)
+		(start 90 125)
+		(end 92 123)
 		(width 1.27)
 		(layer "F.Cu")
@@
 	)
 	(segment
-		(start 82.5 102.5)
-		(end 76 109)
-		(width 0.762)
+		(start 89 116.5)
+		(end 87 116.5)
+		(width 1.27)
 		(layer "F.Cu")
 		(net 26)
 	)
 	(segment
-		(start 92 116)
-		(end 92 123)
+		(start 90 126.5)
+		(end 90 125)
 		(width 1.27)
 		(layer "F.Cu")
@@
 	)
 	(segment
-		(start 90 126.5)
-		(end 92 128.5)
+		(start 92 113.5)
+		(end 92 123)
 		(width 1.27)
 		(layer "F.Cu")
@@
 	)
 	(segment
-		(start 84.88 102.5)
-		(end 88.5 102.5)
+		(start 85 118.5)
+		(end 85 125)
 		(width 1.27)
 		(layer "F.Cu")
@@
 	)
 	(segment
-		(start 92 132.89)
-		(end 92.03 132.92)
+		(start 84.88 102.5)
+		(end 88.5 102.5)
 		(width 1.27)
 		(layer "F.Cu")
@@
 		(polygon
 			(pts
-				(xy 106 113.5) (xy 106 141) (xy 162 141) (xy 162 113.5)
+				(xy 106 114) (xy 106 141.5) (xy 162 141.5) (xy 162 114)
 			)
 		)
